File: project/intv-audio-line-driver.kicad_pcb (KiCad board)
At the start: 2 copper layers, 94 x 67 mm, 22 parts, among them J1 AUD IN, J2 LEFT OUT, J3 RIGHT OUT, J4 +5V IN, J5 GND, Q1 2N3904, Q2 2N3904

Commit message: Add KA358 two-layer routing handoff
Parts:
- removed J5: GND, WirePad_1x01_D3.5mm_Drill1.3mm
- removed R10: 1k, R_Axial_DIN0207_L6.3mm_D2.5mm_P10.16mm_Horizontal
- J1: value AUD IN -> RAW AUD IN
- J2: value LEFT OUT -> BUF AUD OUT
- J3: value RIGHT OUT -> +5V FROM VID
- J4: value +5V IN -> GND FROM VID
- moved J3 81.4 mm to (50.0, 94.0)
- moved J2 6.00 mm to (131.0, 80.0)
- moved J4 6.00 mm to (50.0, 104.0)
- moved R9 6.00 mm to (116.0, 80.0)
- moved J1 4.00 mm to (50.0, 76.0)
Connections:
- net LEFT_OUT renamed AUD_OUT
- J3 pad 1: RIGHT_OUT -> +5V
- J4 pad 1: +5V -> GND
Routing:
- net GND: track 0.00 -> 190.6 mm, vias 0 -> 1
- net +5V: track 0.00 -> 98.0 mm
- net Q1_BASE: track 0.00 -> 84.6 mm
- net Q2_BASE: track 0.00 -> 71.6 mm
- net Q2_EM: track 0.00 -> 44.0 mm
- net Q1_COL: track 0.00 -> 34.3 mm
- net Q2_COL: track 0.00 -> 33.3 mm
- net Q1_EM: track 0.00 -> 30.8 mm
- net AUD_IN: track 0.00 -> 16.0 mm
- net AUDIO_BUS: track 0.00 -> 11.5 mm
- net AUD_OUT: track 0.00 -> 4.84 mm
Other:
- board text added: "+5V FROM VIDEO"
- board text added: "BUFFERED AUDIO OUT"
- board text added: "GND FROM VIDEO"
- board text added: "RAW AUDIO IN"
- board text added: "REV A — ROUTED PROTOTYPE — DO NOT FAB"
- board text removed: "+5V"
- board text removed: "AUD IN"
- board text removed: "GND"
- board text removed: "LEFT OUT"
- board text removed: "REV A — PLACEMENT ONLY — DO NOT FAB"
- board text removed: "RIGHT OUT"
